File: examples/demo_preview/demo_preview.kicad_pcb (KiCad board)
At the start: 2 copper layers, 4 parts, among them U1 XE216-512-TQ128, U2 xs1-a16a-128-fb217, U3 xs1-a8a-64-fb96, U4 XU208-256-TQ64

Commit message: fb236 added.
Parts:
- added U5: XUF216-512-FB236, xmos:FB236, F.Cu at (106.5, 152.0)
